File: HW/MermaidControlUnit/_autosave-STM32.kicad_sch (KiCad schematic)
At the start: 15 parts, among them U1 STM32F103C8Tx, Y1 ABM3-8.000MHZ-D2Y-T, Y2 CM315D

Commit message: folders reorganized, schematic progress
Connections:
- net TX: now reaches U1.42 (PB6)
- net RX: now reaches U1.43 (PB7)
Changed lines of the file:
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@@
+	(wire
+		(pts
+			(xy 143.51 105.41) (xy 129.54 105.41)
+		)
+		(stroke
+			(width 0)
+			(type default)
+		)
+	)
 	(wire
 		(pts
@@
 		(pts
 			(xy 163.83 54.61) (xy 163.83 52.07)
+		)
+		(stroke
+			(width 0)
+			(type default)
+		)
+	)
+	(wire
+		(pts
+			(xy 143.51 107.95) (xy 129.54 107.95)
 		)
 		(stroke
@@
 		)
 	)
+	(label "RX"
+		(at 129.54 107.95 0)
+		(fields_autoplaced yes)
+		(effects
+			(font
+				(size 1.27 1.27)
+			)
+			(justify left bottom)
+		)
+	)
 	(label "OSC32OUT"
 		(at 129.54 85.09 0)
 		(fields_autoplaced yes)
 		(effects
+			(font
+				(size 1.27 1.27)
+			)
+			(justify left bottom)
+		)
+	)
+	(label "TX"
+		(at 129.54 105.41 0)
+		(fields_autoplaced yes)
+		(effects
