File: HW/MermaidControlUnit/levelShifter.kicad_sch (KiCad schematic)
At the start: 0 parts

Commit message: folders reorganized, schematic progress
Parts:
- added C22, C23, C24, C25, C26, C27, C28, C29, C30, C31, C32, C33: 100n, symbol Device:C
- added U3, U5, U6, U7, U8, U9: SN74LVC2T45DCUR, Package_SO:SSOP-8_2.95x2.8mm_P0.65mm, symbol Logic_LevelTranslator:SN74LVC2T45DCUR
Connections:
- new net +3V3: C23.1, C24.1, C26.1, C28.1, C30.1, C32.1, U3.1 (VCCA), U3.5 (DIR), U5.1 (VCCA), U5.5 (DIR), U6.1 (VCCA), U6.5 (DIR), U7.1 (VCCA), U7.5 (DIR), U8.1 (VCCA), U8.5 (DIR), U9.1 (VCCA), U9.5 (DIR)
- new net +5V: C22.1, C25.1, C27.1, C29.1, C31.1, C33.1, U3.8 (VCCB), U5.8 (VCCB), U6.8 (VCCB), U7.8 (VCCB), U8.8 (VCCB), U9.8 (VCCB)
- new net GND: C22.2, C23.2, C24.2, C25.2, C26.2, C27.2, C28.2, C29.2, C30.2, C31.2, C32.2, C33.2, U3.4 (GND), U5.4 (GND), U6.4 (GND), U7.4 (GND), U8.4 (GND), U9.4 (GND)
- new net HVOUT0: U3.7 (B1)
- new net HVOUT1: U3.6 (B2)
- new net HVOUT10: U9.7 (B1)
- new net HVOUT11: U9.6 (B2)
- new net HVOUT2: U5.7 (B1)
- new net HVOUT3: U5.6 (B2)
- new net HVOUT4: U6.7 (B1)
- new net HVOUT5: U6.6 (B2)
- new net HVOUT6: U7.7 (B1)
- new net HVOUT7: U7.6 (B2)
- new net HVOUT8: U8.7 (B1)
- new net HVOUT9: U8.6 (B2)
- new net LVIN0: U3.2 (A1)
- new net LVIN1: U3.3 (A2)
- new net LVIN10: U9.2 (A1)
- new net LVIN11: U9.3 (A2)
- new net LVIN2: U5.2 (A1)
- new net LVIN3: U5.3 (A2)
- new net LVIN4: U6.2 (A1)
- new net LVIN5: U6.3 (A2)
- new net LVIN6: U7.2 (A1)
- new net LVIN7: U7.3 (A2)
- new net LVIN8: U8.2 (A1)
- new net LVIN9: U8.3 (A2)
