File: HW/MermaidControlUnit/outputs.kicad_sch (KiCad schematic)
At the start: 0 parts

Commit message: folders reorganized, schematic progress
Parts:
- added J1, J2, J3, J4, J5, J6: Conn_02x03_RightAngle, Connector_PinHeader_2.54mm:PinHeader_2x03_P2.54mm_Horizontal, symbol Connector_Generic:Conn_02x03_Odd_Even
Connections:
- new net +5V: J1.1 (Pin_1), J1.2 (Pin_2), J2.1 (Pin_1), J2.2 (Pin_2), J3.1 (Pin_1), J3.2 (Pin_2), J4.1 (Pin_1), J4.2 (Pin_2), J5.1 (Pin_1), J5.2 (Pin_2), J6.1 (Pin_1), J6.2 (Pin_2)
- new net GND: J1.5 (Pin_5), J1.6 (Pin_6), J2.5 (Pin_5), J2.6 (Pin_6), J3.5 (Pin_5), J3.6 (Pin_6), J4.5 (Pin_5), J4.6 (Pin_6), J5.5 (Pin_5), J5.6 (Pin_6), J6.5 (Pin_5), J6.6 (Pin_6)
- new net String0: J1.3 (Pin_3)
- new net String1: J1.4 (Pin_4)
- new net String10: J6.3 (Pin_3)
- new net String11: J6.4 (Pin_4)
- new net String2: J2.3 (Pin_3)
- new net String3: J2.4 (Pin_4)
- new net String4: J3.3 (Pin_3)
- new net String5: J3.4 (Pin_4)
- new net String6: J4.3 (Pin_3)
- new net String7: J4.4 (Pin_4)
- new net String8: J5.3 (Pin_3)
- new net String9: J5.4 (Pin_4)
