File: HW/MermaidControlUnit/powering.kicad_sch (KiCad schematic)
At the start: 0 parts

Commit message: folders reorganized, schematic progress
Parts:
- added C1, C2, C5, C6, C7, C8: 22u, symbol Device:C
- added C10, C3, C4, C9: 10u, symbol Device:C
- added C11, C12: 1u, symbol Device:C
- added D1, D2, D3, D4: LED, symbol Device:LED
- added L1: 1uH, symbol Device:L
- added Q1: IRLML6244, Package_TO_SOT_SMD:SOT-23, symbol Transistor_FET:IRLML6244
- added R1: 0R, symbol Device:R
- added R10: 1k, symbol Device:R
- added R11, R12, R13, R14, R2, R3, R4, R5, R6: D.N.P., symbol Device:R
- added R15: 47R, symbol Device:R
- added R16: 10k, symbol Device:R
- added R17: 100k, symbol Device:R
- added R7: 82k, symbol Device:R
- added R8: NTC 100k, symbol Device:R
- added R9: 2R, symbol Device:R
- added U2: IP5310, Package_DFN_QFN:QFN-32-1EP_5x5mm_P0.5mm_EP3.3x3.3mm_ThermalVias, symbol library:IP5310
- added U4: AP2112K-3.3, Package_TO_SOT_SMD:SOT-23-5, symbol Regulator_Linear:AP2112K-3.3
Connections:
- new net: R3.1, R4.1, U2.3 (VSET)
- new net: Q1.1 (G), R15.1, R16.2
- new net: R7.1, R8.1, U2.6 (NTC)
- new net: D1.1 (K), D2.2 (A), R13.1, U2.1 (L2/SDA)
- new net: R10.1, R11.1, U2.2 (L3/IRQ)
- new net: D1.2 (A), D2.1 (K), D3.2 (A), D4.1 (K), R10.2
- new net: C4.1, R9.1
- new net: C2.1, R1.1, U2.9 (BAT)
- new net: R5.1, R6.1, U2.4 (VTHS)
- new net: L1.1, U2.14 (LX), U2.15 (LX), U2.16 (LX), U2.17 (LX), U2.18 (LX)
- new net: D3.1 (K), D4.2 (A), R12.1, U2.32 (L1/SCK)
- new net: R2.1, U2.5 (RSET)
- new net: Q1.3 (D), R14.1, U2.8 (KEY)
- new net +3V3: C10.1, C12.1, U4.5 (VOUT)
- new net +5V: C5.1, C6.1, C7.1, C8.1, U2.19 (VOUT), U2.20 (VOUT), U2.21 (VOUT), U2.22 (VOUT)
- new net +BATT: C1.1, C11.1, C9.1, L1.2, R1.2, R14.2, R3.2, R5.2, U4.1 (VIN)
- new net +VIN: C3.1, R9.2, U2.23 (VIN), U2.24 (VIN)
- new net GND: C1.2, C10.2, C11.2, C12.2, C2.2, C3.2, C4.2, C5.2, C6.2, C7.2, C8.2, C9.2, Q1.2 (S), R16.1, R17.1, R2.2, R4.2, R6.2, R7.2, R8.2, U2.33 (EPAD), U2.7 (AGND), U4.2 (GND)
- new net IRQ: R11.2
- new net KEY: R15.2
- new net LDO_EN: R17.2, U4.3 (EN)
- new net SCK: R12.2
- new net SDA: R13.2
- no-connect marks 0 -> 1
