File: HW/MermaidControlUnit_A/MermaidControlUnit.kicad_pcb (KiCad board)
At the start: 2 copper layers, 163 parts, among them J1 Conn_01x05, J10 Conn_02x03_RightAngle, J11 Conn_02x03_RightAngle, J12 Coil_1, J13 Coil_2, J2 Conn_01x03, J3 Conn_01x03, J4 Batt+, J5 Batt-, J6 Conn_02x03_RightAngle, J7 Conn_02x03_RightAngle, J8 Conn_02x03_RightAngle, J9 Conn_02x03_RightAngle, Q1 IRLML6244, U1 STM32F103C8Tx, U10 BQ51013C-Q1, U2 AP2112K-3.3, U3 IP5310, U4 SN74LVC2T45DCUR, U5 SN74LVC2T45DCUR, U6 SN74LVC2T45DCUR, U7 SN74LVC2T45DCUR, U8 SN74LVC2T45DCUR, U9 SN74LVC2T45DCUR, Y1 ABM3-8.000MHZ-D2Y-T, Y2 CM315D

Commit message: hw progress
Parts:
- added C55: 1u, Capacitor_SMD:C_0603_1608Metric, F.Cu at (246.8, 83.5)
- added C56: 10u, Capacitor_SMD:C_0603_1608Metric, F.Cu at (248.5, 83.5)
- added C57: 1u, Capacitor_SMD:C_0603_1608Metric, F.Cu at (240.5, 83.5)
- added C58: 47u, Capacitor_SMD:C_0805_2012Metric, F.Cu at (201.8, 75.5)
- added C59: 47u, Capacitor_SMD:C_0805_2012Metric, F.Cu at (201.8, 77.8)
- added C60: 47u, Capacitor_SMD:C_0805_2012Metric, F.Cu at (211.6, 54.8)
- added C61: 47u, Capacitor_SMD:C_0805_2012Metric, F.Cu at (211.5, 57.0)
- added R38: D.N.P., Resistor_SMD:R_0603_1608Metric, F.Cu at (227.0, 75.2)
- added U11: NCP45520, Package_DFN_QFN:DFN-8-1EP_2x2mm_P0.5mm_EP1.05x1.75mm, F.Cu at (244.2, 83.4)
- L1: footprint Inductor_SMD:L_Sunlord_MWSA1204S-1R0 -> Inductor_SMD:L_PCC-M1040M-LP
- TP1, TP10, TP11, TP12, TP13, TP14, TP15, TP16, TP17, TP18, TP19, TP2, TP20, TP21, TP22, TP23, TP24, TP25, TP26, TP27, TP28, TP29, TP3, TP30, TP31, TP32, TP33, TP34, TP35, TP36, TP4, TP5, TP6, TP7, TP8, TP9: footprint TestPoint:TestPoint_Pad_D2.0mm -> TestPoint:TestPoint_Pad_D1.5mm
- moved R25 69.3 mm to (220.2, 73.5), turned to 180 degrees
- moved R23 66.8 mm to (220.2, 75.2), turned to 0 degrees
- moved R24 63.2 mm to (217.8, 78.5), turned to 90 degrees
- moved Q1 62.5 mm to (220.2, 78.2), turned to -90 degrees
- moved J4 60.1 mm to (204.0, 84.0), turned to 90 degrees
- moved R22 58.4 mm to (220.2, 81.2), turned to 0 degrees
- moved F1 54.5 mm to (202.0, 81.5), turned to 180 degrees
- moved J5 53.4 mm to (198.0, 84.0), turned to 90 degrees
- moved R29 51.7 mm to (218.0, 60.8)
- moved TP26 50.9 mm to (215.8, 84.0), turned to -90 degrees
- moved TP21 48.6 mm to (225.0, 75.8)
- moved TP29 48.0 mm to (216.2, 55.2), turned to 90 degrees
- moved TP1 47.5 mm to (223.0, 74.2)
- moved R1 46.6 mm to (223.0, 78.8)
- moved D1 46.6 mm to (226.0, 78.8)
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Connections:
- J10 pad 1: +5V -> +5V_SW
- J10 pad 2: +5V -> +5V_SW
- J11 pad 1: +5V -> +5V_SW
- J11 pad 2: +5V -> +5V_SW
- J6 pad 1: +5V -> +5V_SW
- J6 pad 2: +5V -> +5V_SW
- J7 pad 1: +5V -> +5V_SW
- J7 pad 2: +5V -> +5V_SW
- J8 pad 1: +5V -> +5V_SW
- J8 pad 2: +5V -> +5V_SW
- J9 pad 1: +5V -> +5V_SW
- J9 pad 2: +5V -> +5V_SW
- TP10 pad 1: /STM32/TIM3_CH1 -> /STM32/TIM4_CH2
- TP11 pad 1: /STM32/TIM4_CH3 -> /STM32/TIM3_CH2
- TP12 pad 1: /STM32/TIM3_CH2 -> /STM32/TIM4_CH1
- TP13 pad 1: /STM32/TIM4_CH4 -> /STM32/TIM3_CH1
- TP2 pad 1: /STM32/TIM2_CH1 -> /STM32/TIM2_CH4
- TP3 pad 1: /STM32/TIM3_CH3 -> /STM32/TIM2_CH2
- TP4 pad 1: /STM32/TIM2_CH2 -> /STM32/TIM2_CH3
- TP5 pad 1: /STM32/TIM3_CH4 -> /STM32/TIM2_CH1
- TP6 pad 1: /STM32/TIM2_CH3 -> /STM32/TIM4_CH4
- TP7 pad 1: /STM32/TIM4_CH1 -> /STM32/TIM3_CH4
- TP8 pad 1: /STM32/TIM2_CH4 -> /STM32/TIM4_CH3
- TP9 pad 1: /STM32/TIM4_CH2 -> /STM32/TIM3_CH3
- U1 pad 41: unconnected-(U1-PB5-Pad41) -> /STM32/+5V_EN
- U4 pad 2: /STM32/TIM2_CH1 -> /STM32/TIM2_CH4
- U4 pad 3: /STM32/TIM2_CH2 -> /STM32/TIM2_CH3
- U5 pad 2: /STM32/TIM3_CH3 -> /STM32/TIM2_CH2
- U5 pad 3: /STM32/TIM3_CH4 -> /STM32/TIM2_CH1
- U6 pad 2: /STM32/TIM2_CH3 -> /STM32/TIM4_CH4
- U6 pad 3: /STM32/TIM2_CH4 -> /STM32/TIM4_CH3
- U7 pad 2: /STM32/TIM4_CH1 -> /STM32/TIM3_CH4
- U7 pad 3: /STM32/TIM4_CH2 -> /STM32/TIM3_CH3
- U8 pad 2: /STM32/TIM3_CH1 -> /STM32/TIM4_CH2
- U8 pad 3: /STM32/TIM3_CH2 -> /STM32/TIM4_CH1
- U9 pad 2: /STM32/TIM4_CH3 -> /STM32/TIM3_CH2
- U9 pad 3: /STM32/TIM4_CH4 -> /STM32/TIM3_CH1
Routing:
- net +3V3: track 0.00 -> 199.0 mm, vias 0 -> 15
- net +5V: track 0.00 -> 136.4 mm, vias 0 -> 4
- net +5V_SW: track 0.00 -> 98.3 mm, vias 0 -> 2
- net +BATT: track 0.00 -> 91.1 mm, vias 0 -> 6
- net /STM32/TIM2_CH4: track 0.00 -> 44.9 mm
- net /STM32/TIM3_CH1: track 0.00 -> 44.0 mm
- net /STM32/TIM2_CH3: track 0.00 -> 40.5 mm
- net /STM32/TIM3_CH2: track 0.00 -> 40.3 mm
- net /Wireless Charging/+5V_Charging: track 6.35 -> 45.9 mm
- net Net-(Q1-D): track 0.00 -> 36.9 mm, vias 0 -> 4
- net /STM32/TIM3_CH3: track 0.00 -> 36.7 mm
- net /STM32/TIM3_CH4: track 0.00 -> 36.5 mm
- net /STM32/+5VSense: track 0.00 -> 36.4 mm
- net /STM32/IR_Receiver: track 0.00 -> 34.5 mm, vias 0 -> 1
- net /STM32/+VbattSense: track 0.00 -> 30.7 mm
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- added copper zone on F.Cu, net +3V3
- added copper zone on F.Cu, net +5V
- added copper zone on F.Cu, net +5V_SW
- added copper zone on B.Cu, net +BATT
- added copper zone on F.Cu, net +BATT
- added copper zone on F.Cu, net /Wireless Charging/+5V_Charging
- added copper zone on B.Cu, net GND
- added copper zone on F.Cu, net GND
- added copper zone on B.Cu, net Net-(J12-Pin_1)
- added copper zone on F.Cu, net Net-(J12-Pin_1)
- added copper zone on B.Cu, net Net-(J13-Pin_1)
- added copper zone on F.Cu, net Net-(J13-Pin_1)
- added copper zone on B.Cu, net Net-(L1-Pad1)
- added copper zone on F.Cu, net Net-(L1-Pad1)
- added copper zone on B.Cu, net Net-(U10-AC1)
- added copper zone on F.Cu, net Net-(U10-AC1)
- added copper zone on F.Cu, net Net-(U10-RECT)
Other:
- board outline added: 75 x 70 mm

Commit message: hw progress
Parts:
- added G***: LOGO, Library:AuroraSymbol10mm, F.Cu at (192.4, 32.2)
- added R39: D.N.P., Resistor_SMD:R_0603_1608Metric, F.Cu at (244.2, 82.0)
- J1: footprint Connector_PinHeader_2.54mm:PinHeader_1x05_P2.54mm_Horizontal -> Library:PinHeader_1x05_P2.54mm_Horizontal_SmallSilk
- J10, J11, J6, J7, J8, J9: footprint Connector_PinHeader_2.54mm:PinHeader_2x03_P2.54mm_Horizontal -> Library:PinHeader_2x03_P2.54mm_Horizontal_SmallSilk
- J2, J3: footprint Connector_PinHeader_2.54mm:PinHeader_1x03_P2.54mm_Horizontal -> Library:PinHeader_1x03_P2.54mm_Horizontal_SmallSilk
- moved C55 0.75 mm to (246.8, 84.2)
- moved C56 0.75 mm to (248.5, 84.2)
- moved C57 0.75 mm to (240.5, 84.2)
- moved U11 0.75 mm to (244.2, 84.2)
Routing:
- net +5V: track 136.4 -> 134.0 mm
- net +5V_SW: track 98.3 -> 96.3 mm
- net GND: track 1.84 -> 0.00 mm
- net /STM32/+5V_EN: track 28.4 -> 27.4 mm
Other:
- board size 75 x 70 mm -> 78.1 x 69 mm
- board text added: "+"
- board text added: "+3V3"
- board text added: "+5V"
- board text added: "-"
- board text added: "01/24"
- board text added: "25% 50% 75% 100%"
- board text added: "BATT Li-3.7V"
- board text added: "DATA"
- board text added: "GND"
- board text added: "IR RECEIVER"
- board text added: "LED STRINGS"
- board text added: "Mermaid Control Unit"
- board text added: "PROGRAMMING"
- board text added: "QI CHARGING INDUCTOR"
- board text added: "RX"
- board text added: "Rev. A"
- board text added: "SWCLK"
- board text added: "SWDIO"
- board text added: "String0&1"
- board text added: "String10&11"
- board text added: "String2&3"
- board text added: "String4&5"
- board text added: "String6&7"
- board text added: "String8&9"
- board text added: "StringTOP&BOT"
- board text added: "TX"
- board text added: "UART"
- board text added: "~{RST}"

Commit message: production rev A
Parts:
- added R40: 30k, Resistor_SMD:R_0603_1608Metric, F.Cu at (219.8, 40.8)
- C36: value 10n -> 68n
- C37: value 10n -> 47n
- C38: value 10n -> 39n
- C39: value 100n -> 2n2
- C40: value 100n -> 100p
- D2, D8: value LED -> RED
- D3: value LED -> GREEN
- D4, D5, D6, D7: value LED -> BLUE
- R25: value 220R -> 110R
- R33: value 10k -> 110R
- R34: value NTC -> NTC 100k
- U1: value STM32F103C8Tx -> STM32F103CBTx
- U3: footprint Package_DFN_QFN:QFN-32-1EP_5x5mm_P0.5mm_EP3.3x3.3mm_ThermalVias -> Package_DFN_QFN:QFN-32-1EP_5x5mm_P0.5mm_EP3.6x3.6mm_ThermalVias
- U4, U5, U6, U7, U8, U9: value SN74LVC2T45DCUR -> SN74LVC2T45DCTR
- moved TP32 4.96 mm to (222.8, 36.5)
- moved C57 0.18 mm to (240.5, 84.1)
Routing:
- net Net-(U10-ILIM): track 12.3 -> 17.0 mm
- net +3V3: track 199.0 -> 202.3 mm
- net unconnected-(U3-DPA-Pad28): track 0.00 -> 2.48 mm
- net unconnected-(U3-DMA-Pad27): track 0.00 -> 2.48 mm
- net +5V: track 134.0 -> 136.2 mm
- net Net-(U10-TS/CTRL): track 18.0 -> 19.8 mm
- net +BATT: track 91.1 -> 92.1 mm, vias 6 -> 20
- net +5V_SW: track 96.3 -> 96.8 mm
- net Net-(U10-AC1): vias 1 -> 11
- net Net-(L1-Pad1): vias 1 -> 15
- net Net-(J13-Pin_1): vias 0 -> 18
- net Net-(J12-Pin_1): vias 0 -> 10
- net GND: vias 73 -> 74
