File: HW/MermaidControlUnit_A/STM32.kicad_sch (KiCad schematic)
At the start: 15 parts, among them U1 STM32F103C8Tx, Y1 ABM3-8.000MHZ-D2Y-T, Y2 CM315D

Commit message: pinmapping
Connections:
- net RX: now also U1.31 (PA10); no longer U1.43 (PB7)
- net TX: now also U1.30 (PA9); no longer U1.42 (PB6)
- net IR_Receiver: now reaches U1.10 (PA0)
- net IR_Receiver: now also U1.11 (PA1)
- net TIM2_CH3: now reaches U1.12 (PA2)
- net TIM2_CH4: now reaches U1.13 (PA3)
- net TIM3_CH1: now reaches U1.16 (PA6)
- net TIM3_CH2: now reaches U1.17 (PA7)
- net TIM3_CH3: now reaches U1.18 (PB0)
- net TIM3_CH4: now reaches U1.19 (PB1)
- net IRQ_Boost: now reaches U1.20 (PB2)
- net I2C2_SCL: now reaches U1.21 (PB10)
- net I2C2_SDA: now reaches U1.22 (PB11)
- net TIM2_CH1: now reaches U1.38 (PA15)
- net TIM2_CH2: now reaches U1.39 (PB3)
- net TIM4_CH3: now reaches U1.45 (PB8)
- net TIM4_CH4: now reaches U1.46 (PB9)
- new net TIM4_CH1: U1.42 (PB6)
- new net TIM4_CH2: U1.43 (PB7)

Commit message: HW design progress
Parts:
- added C10, C11: 100n, Capacitor_SMD:C_0603_1608Metric, symbol Device:C
- added D2, D3: LED, LED_SMD:LED_0603_1608Metric, symbol Device:LED
- added J1: Conn_01x05, Connector_PinHeader_2.54mm:PinHeader_1x05_P2.54mm_Horizontal, symbol Connector_Generic:Conn_01x05
- added J2, J3: Conn_01x03, Connector_PinHeader_2.54mm:PinHeader_1x03_P2.54mm_Horizontal, symbol Connector_Generic:Conn_01x03
- added R10, R11, R8, R9: 100k, Resistor_SMD:R_0603_1608Metric, symbol Device:R
- added R2, R3: 470R, Resistor_SMD:R_0603_1608Metric, symbol Device:R
- added R6: 10k, Resistor_SMD:R_0603_1608Metric, symbol Device:R
- added TP14, TP15, TP16, TP17, TP18, TP19, TP20: TestPoint, TestPoint:TestPoint_Pad_D2.0mm, symbol Connector:TestPoint
- C1: renamed from C18; footprint (none) -> Capacitor_SMD:C_0603_1608Metric
- C2: renamed from C20; footprint (none) -> Capacitor_SMD:C_0603_1608Metric
- C3: renamed from C19; footprint (none) -> Capacitor_SMD:C_0603_1608Metric
- C4: renamed from C21; footprint (none) -> Capacitor_SMD:C_0603_1608Metric
- C5: renamed from C17; footprint (none) -> Capacitor_SMD:C_0603_1608Metric
- C6: renamed from C16; footprint (none) -> Capacitor_SMD:C_0603_1608Metric
- C7: renamed from C15; footprint (none) -> Capacitor_SMD:C_0603_1608Metric
- C8: renamed from C14; footprint (none) -> Capacitor_SMD:C_0603_1608Metric
- C9: renamed from C13; footprint (none) -> Capacitor_SMD:C_0603_1608Metric
- R4: renamed from R20; footprint (none) -> Resistor_SMD:R_0603_1608Metric
- R5: renamed from R19; footprint (none) -> Resistor_SMD:R_0603_1608Metric
- R7: renamed from R18; footprint (none) -> Resistor_SMD:R_0603_1608Metric
Connections:
- net +3V3: now also J1.5 (Pin_5), J3.3 (Pin_3), R6.2
- net GND: now also C10.2, C11.2, D2.1 (K), D3.1 (K), J1.3 (Pin_3), J2.3 (Pin_3), J3.2 (Pin_2), R11.1, R9.1
- net IR_Receiver: now also J3.1 (Pin_1), TP19.1
- net RX: now also J2.2 (Pin_2)
- net SWCLK: now also J1.2 (Pin_2)
- net SWDIO: now also J1.1 (Pin_1)
- net TX: now also J2.1 (Pin_1)
- net nRST: now also J1.4 (Pin_4), R6.1, TP14.1
- net at R5.2, U1.44 (BOOT0): now also TP15.1
- net +5VSense: now reaches U1.14 (PA4)
- net +5VSense: now also C10.1, R8.1, R9.2, TP18.1
- net +VbattSense: now reaches U1.15 (PA5)
- net +VbattSense: now also C11.1, R10.1, R11.2, TP20.1
- net LED1: now reaches U1.2 (PC13)
- net LED1: now also R2.1
- net boostWkUp: now reaches U1.25 (PB12)
- net powerOn: now reaches U1.26 (PB13)
- net at U1.32 (PA11): now also TP16.1
- net at U1.33 (PA12): now also TP17.1
- net LED2: now reaches U1.40 (PB4)
- net LED2: now also R3.1
- new net: D2.2 (A), R2.2
- new net: D3.2 (A), R3.2
- new net +5V: R8.2
- new net +BATT: R10.2
- no-connect marks 0 -> 4
Other:
- moved on the sheet: R5, R7

Commit message: hw progress
Parts:
- TP14, TP15, TP16, TP17, TP18, TP19, TP20: footprint TestPoint:TestPoint_Pad_D2.0mm -> TestPoint:TestPoint_Pad_D1.5mm
Connections:
- net +5V_EN: now reaches U1.41 (PB5)
- no-connect marks 4 -> 3
Changed lines of the file:
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@@
 		(at 179.07 82.55)
 	)
-	(no_connect
-		(at 143.51 102.87)
-	)
 	(wire
 		(pts
@@
 	(wire
 		(pts
+			(xy 129.54 102.87) (xy 143.51 102.87)
+		)
+		(stroke
+			(width 0)
+			(type default)
+		)
+	)
+	(wire
+		(pts
 			(xy 236.22 68.58) (xy 236.22 72.39)
 		)
@@
 		)
 	)
+	(label "+5V_EN"
+		(at 129.54 102.87 0)
+		(fields_autoplaced yes)
+		(effects
+			(font
+				(size 1.27 1.27)
+			)
+			(justify left bottom)
+		)
+	)
 	(label "OSC32OUT"
 		(at 129.54 85.09 0)
@@
 		)
 	)
+	(hierarchical_label "+5V_EN"
+		(shape output)
+		(at 129.54 102.87 180)
+		(fields_autoplaced yes)
+		(effects
+			(font
+				(size 1.27 1.27)
+			)
+			(justify right)
+		)
+	)
 	(hierarchical_label "TIM4_CH4"
 		(shape output)
@@
 			)
 		)
-		(property "Footprint" "TestPoint:TestPoint_Pad_D2.0mm"
+		(property "Footprint" "TestPoint:TestPoint_Pad_D1.5mm"
 			(at 196.85 95.25 0)
 			(effects
@@
 			)
 		)
-		(property "Footprint" "TestPoint:TestPoint_Pad_D2.0mm"
+		(property "Footprint" "TestPoint:TestPoint_Pad_D1.5mm"
 			(at 132.08 67.31 0)
 			(effects
@@
 			)
 		)
-		(property "Footprint" "TestPoint:TestPoint_Pad_D2.0mm"
+		(property "Footprint" "TestPoint:TestPoint_Pad_D1.5mm"
 			(at 247.65 74.93 0)
 			(effects
@@
 			)
 		)
-		(property "Footprint" "TestPoint:TestPoint_Pad_D2.0mm"
+		(property "Footprint" "TestPoint:TestPoint_Pad_D1.5mm"
 			(at 196.85 97.79 0)
 			(effects
@@
 			)
 		)
-		(property "Footprint" "TestPoint:TestPoint_Pad_D2.0mm"
+		(property "Footprint" "TestPoint:TestPoint_Pad_D1.5mm"
 			(at 241.3 30.48 0)
 			(effects
@@
 			)
 		)
-		(property "Footprint" "TestPoint:TestPoint_Pad_D2.0mm"
+		(property "Footprint" "TestPoint:TestPoint_Pad_D1.5mm"
 			(at 128.27 57.15 0)
 			(effects
@@
 			)
 		)
-		(property "Footprint" "TestPoint:TestPoint_Pad_D2.0mm"
+		(property "Footprint" "TestPoint:TestPoint_Pad_D1.5mm"
 			(at 229.87 72.39 0)
 			(effects

Commit message: hw progress
Parts:
- J1: footprint Connector_PinHeader_2.54mm:PinHeader_1x05_P2.54mm_Horizontal -> Library:PinHeader_1x05_P2.54mm_Horizontal_SmallSilk
- J2, J3: footprint Connector_PinHeader_2.54mm:PinHeader_1x03_P2.54mm_Horizontal -> Library:PinHeader_1x03_P2.54mm_Horizontal_SmallSilk
Changed lines of the file:
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@@
 			)
 		)
-		(property "Footprint" "Connector_PinHeader_2.54mm:PinHeader_1x05_P2.54mm_Horizontal"
+		(property "Footprint" "Library:PinHeader_1x05_P2.54mm_Horizontal_SmallSilk"
 			(at 251.46 113.03 0)
 			(effects
@@
 			)
 		)
-		(property "Footprint" "Connector_PinHeader_2.54mm:PinHeader_1x03_P2.54mm_Horizontal"
+		(property "Footprint" "Library:PinHeader_1x03_P2.54mm_Horizontal_SmallSilk"
 			(at 251.46 133.35 0)
 			(effects
@@
 			)
 		)
-		(property "Footprint" "Connector_PinHeader_2.54mm:PinHeader_1x03_P2.54mm_Horizontal"
+		(property "Footprint" "Library:PinHeader_1x03_P2.54mm_Horizontal_SmallSilk"
 			(at 254 35.56 0)
 			(effects

Commit message: production rev A
Parts:
- removed U1: STM32F103C8Tx, Package_QFP:LQFP-48_7x7mm_P0.5mm, symbol MCU_ST_STM32F1:STM32F103C8Tx
- added U1: STM32F103CBTx, Package_QFP:LQFP-48_7x7mm_P0.5mm, symbol MCU_ST_STM32F1:STM32F103CBTx
- C1, C2, C3, C4: Part Number (none) -> GCM1885C1H200JA16D
- C10, C11, C5, C6, C7, C8: Part Number (none) -> CC0603KRX7R9BB104
- C9: Part Number (none) -> CL10A106MA8NRNC
- D2: value LED -> RED; Part Number (none) -> APT1608EC
- D3: value LED -> GREEN; Part Number (none) -> APT1608CGCK
- J1: Part Number (none) -> 5AMW4-10560-105-W0
- J2, J3: Part Number (none) -> X6511WR-03H-C60D30R2
- R10, R11, R8, R9: Part Number (none) -> RC0603FR-07100KL
- R2, R3: Part Number (none) -> RC0603FR-07470RL
- R4: Part Number (none) -> RC0603FR-071ML
- R5, R7: Part Number (none) -> RC0603FR-070RL
- R6: Part Number (none) -> RC0603FR-0710KL
- Y1: Part Number (none) -> ABM3-8.000MHZ-D2Y-T
- Y2: Part Number (none) -> CM315D32768DZFT
Connections:
- net +3V3: now also U1.24 (VDD), U1.36 (VDD), U1.48 (VDD), U1.9 (VDDA)
- net +5VSense: now also U1.14 (PA4)
- net +5V_EN: now also U1.41 (PB5)
- net +VbattSense: now also U1.15 (PA5)
- net GND: now also U1.23 (VSS), U1.35 (VSS), U1.47 (VSS), U1.8 (VSSA)
- net I2C2_SCL: now also U1.21 (PB10)
- net I2C2_SDA: now also U1.22 (PB11)
- net IRQ_Boost: now also U1.20 (PB2)
- net IR_Receiver: now also U1.10 (PA0), U1.11 (PA1)
- net LED1: now also U1.2 (PC13)
- net LED2: now also U1.40 (PB4)
- net OSC32IN: now also U1.3 (PC14)
- net OSC32OUT: now also U1.4 (PC15)
- net OSCIN: now also U1.5 (PD0)
- net OSCOUT: now also U1.6 (PD1)
- net RX: now also U1.31 (PA10)
- net SWCLK: now also U1.37 (PA14)
- net SWDIO: now also U1.34 (PA13)
- net TIM2_CH1: now also U1.38 (PA15)
- net TIM2_CH2: now also U1.39 (PB3)
- net TIM2_CH3: now also U1.12 (PA2)
- net TIM2_CH4: now also U1.13 (PA3)
- net TIM3_CH1: now also U1.16 (PA6)
- net TIM3_CH2: now also U1.17 (PA7)
- net TIM3_CH3: now also U1.18 (PB0)
- net TIM3_CH4: now also U1.19 (PB1)
- net TIM4_CH1: now also U1.42 (PB6)
- net TIM4_CH2: now also U1.43 (PB7)
- net TIM4_CH3: now also U1.45 (PB8)
- net TIM4_CH4: now also U1.46 (PB9)
- net TX: now also U1.30 (PA9)
- net boostWkUp: now also U1.25 (PB12)
- net nRST: now also U1.7 (NRST)
- net powerOn: now also U1.26 (PB13)
- net at R5.2, TP15.1: now also U1.44 (BOOT0)
- net at TP16.1: now also U1.32 (PA11)
- net at R7.2: now also U1.1 (VBAT)
- net at TP17.1: now also U1.33 (PA12)
