File: HW/MermaidControlUnit_A/levelShifter.kicad_sch (KiCad schematic)
At the start: 18 parts, among them U3 SN74LVC2T45DCUR, U5 SN74LVC2T45DCUR, U6 SN74LVC2T45DCUR, U7 SN74LVC2T45DCUR, U8 SN74LVC2T45DCUR, U9 SN74LVC2T45DCUR

Commit message: HW design progress
Parts:
- C24: renamed from C23; footprint (none) -> Capacitor_SMD:C_0603_1608Metric
- C25: renamed from C28; footprint (none) -> Capacitor_SMD:C_0603_1608Metric
- C26: renamed from C22; footprint (none) -> Capacitor_SMD:C_0603_1608Metric
- C27: renamed from C29; footprint (none) -> Capacitor_SMD:C_0603_1608Metric
- C28: renamed from C24; footprint (none) -> Capacitor_SMD:C_0603_1608Metric
- C29: renamed from C30; footprint (none) -> Capacitor_SMD:C_0603_1608Metric
- C30: renamed from C25; footprint (none) -> Capacitor_SMD:C_0603_1608Metric
- C31: footprint (none) -> Capacitor_SMD:C_0603_1608Metric
- C32: renamed from C26; footprint (none) -> Capacitor_SMD:C_0603_1608Metric
- C33: renamed from C32; footprint (none) -> Capacitor_SMD:C_0603_1608Metric
- C34: renamed from C27; footprint (none) -> Capacitor_SMD:C_0603_1608Metric
- C35: renamed from C33; footprint (none) -> Capacitor_SMD:C_0603_1608Metric
- renumbered U3 to U4, U7 to U5, U5 to U6, U8 to U7, U6 to U8

Commit message: production rev A
Parts:
- C24, C25, C26, C27, C28, C29, C30, C31, C32, C33, C34, C35: Part Number (none) -> CC0603KRX7R9BB104
- U4, U5, U6, U7, U8, U9: value SN74LVC2T45DCUR -> SN74LVC2T45DCTR; Part Number (none) -> SN74LVC2T45DCTR
Changed lines of the file:
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@@
 			)
 		)
+		(property "Part Number" "CC0603KRX7R9BB104"
+			(at 232.41 105.41 0)
+			(effects
+				(font
+					(size 1.27 1.27)
+				)
+				(hide yes)
+			)
+		)
 		(pin "2"
 		)
@@
 			)
 		)
-		(property "Value" "SN74LVC2T45DCUR"
+		(property "Value" "SN74LVC2T45DCTR"
 			(at 146.9741 78.74 0)
 			(effects
@@
 			)
 		)
+		(property "Part Number" "SN74LVC2T45DCTR"
+			(at 144.78 63.5 0)
+			(effects
+				(font
+					(size 1.27 1.27)
+				)
+				(hide yes)
+			)
+		)
 		(pin "7"
 		)
@@
 			)
 		)
+		(property "Part Number" "CC0603KRX7R9BB104"
+			(at 54.61 44.45 0)
+			(effects
+				(font
+					(size 1.27 1.27)
+				)
+				(hide yes)
+			)
+		)
 		(pin "2"
 		)
@@
 			)
 		)
-		(property "Value" "SN74LVC2T45DCUR"
+		(property "Value" "SN74LVC2T45DCTR"
 			(at 68.2341 139.7 0)
 			(effects
@@
 			)
 		)
+		(property "Part Number" "SN74LVC2T45DCTR"
+			(at 66.04 124.46 0)
+			(effects
+				(font
+					(size 1.27 1.27)
+				)
+				(hide yes)
+			)
+		)
 		(pin "7"
 		)
@@
 			)
 		)
+		(property "Part Number" "CC0603KRX7R9BB104"
+			(at 77.47 105.41 0)
+			(effects
+				(font
+					(size 1.27 1.27)
+				)
+				(hide yes)
+			)
+		)
 		(pin "2"
 		)
@@
 			)
 		)
+		(property "Part Number" "CC0603KRX7R9BB104"
+			(at 209.55 105.41 0)
+			(effects
+				(font
+					(size 1.27 1.27)
+				)
+				(hide yes)
+			)
+		)
 		(pin "2"
 		)
@@
 			)
 		)
+		(property "Part Number" "CC0603KRX7R9BB104"
+			(at 77.47 44.45 0)
+			(effects
+				(font
+					(size 1.27 1.27)
+				)
+				(hide yes)
+			)
+		)
 		(pin "2"
 		)
@@
 			)
 		)
-		(property "Value" "SN74LVC2T45DCUR"
+		(property "Value" "SN74LVC2T45DCTR"
 			(at 146.9741 139.7 0)
 			(effects
@@
 			)
 		)
+		(property "Part Number" "SN74LVC2T45DCTR"
+			(at 144.78 124.46 0)
+			(effects
+				(font
+					(size 1.27 1.27)
+				)
+				(hide yes)
+			)
+		)
 		(pin "7"
 		)
@@
 			)
 		)
-		(property "Value" "SN74LVC2T45DCUR"
+		(property "Value" "SN74LVC2T45DCTR"
 			(at 223.1741 139.7 0)
 			(effects
@@
 			)
 		)
+		(property "Part Number" "SN74LVC2T45DCTR"
+			(at 220.98 124.46 0)
+			(effects
+				(font
+					(size 1.27 1.27)
+				)
+				(hide yes)
+			)
+		)
 		(pin "7"
 		)
@@
 			)
 		)
+		(property "Part Number" "CC0603KRX7R9BB104"
+			(at 133.35 44.45 0)
+			(effects
+				(font
+					(size 1.27 1.27)
+				)
+				(hide yes)
+			)
+		)
 		(pin "2"
 		)
@@
 			)
 		)
+		(property "Part Number" "CC0603KRX7R9BB104"
+			(at 156.21 44.45 0)
+			(effects
+				(font
+					(size 1.27 1.27)
+				)
+				(hide yes)
+			)
+		)
 		(pin "2"
 		)
@@
 			)
 		)
+		(property "Part Number" "CC0603KRX7R9BB104"
+			(at 209.55 44.45 0)
+			(effects
+				(font
+					(size 1.27 1.27)
+				)
+				(hide yes)
+			)
+		)
 		(pin "2"
 		)
@@
 			)
 		)
-		(property "Value" "SN74LVC2T45DCUR"
+		(property "Value" "SN74LVC2T45DCTR"
 			(at 223.1741 78.74 0)
 			(effects
@@
 			)
 		)
+		(property "Part Number" "SN74LVC2T45DCTR"
+			(at 220.98 63.5 0)
+			(effects
+				(font
+					(size 1.27 1.27)
+				)
+				(hide yes)
+			)
+		)
 		(pin "7"
 		)
@@
 			)
 		)
+		(property "Part Number" "CC0603KRX7R9BB104"
+			(at 156.21 105.41 0)
+			(effects
+				(font
+					(size 1.27 1.27)
+				)
+				(hide yes)
+			)
+		)
 		(pin "2"
 		)
@@
 			)
 		)
-		(property "Value" "SN74LVC2T45DCUR"
+		(property "Value" "SN74LVC2T45DCTR"
 			(at 68.2341 78.74 0)
 			(effects
@@
 			)
 		)
+		(property "Part Number" "SN74LVC2T45DCTR"
+			(at 66.04 63.5 0)
+			(effects
+				(font
+					(size 1.27 1.27)
+				)
+				(hide yes)
+			)
+		)
 		(pin "7"
 		)
@@
 			)
 		)
+		(property "Part Number" "CC0603KRX7R9BB104"
+			(at 133.35 105.41 0)
+			(effects
+				(font
+					(size 1.27 1.27)
+				)
+				(hide yes)
+			)
+		)
 		(pin "2"
 		)
@@
 			)
 		)
+		(property "Part Number" "CC0603KRX7R9BB104"
+			(at 54.61 105.41 0)
+			(effects
+				(font
+					(size 1.27 1.27)
+				)
+				(hide yes)
+			)
+		)
 		(pin "2"
 		)
@@
 			(at 232.41 44.45 0)
 			(effects
+				(font
+					(size 1.27 1.27)
+				)
+				(hide yes)
+			)
+		)
+		(property "Part Number" "CC0603KRX7R9BB104"
+			(at 232.41 44.45 0)
+			(effects
