File: HW/MermaidControlUnit_A/outputs.kicad_sch (KiCad schematic)
At the start: 6 parts, among them J1 Conn_02x03_RightAngle, J2 Conn_02x03_RightAngle, J3 Conn_02x03_RightAngle, J4 Conn_02x03_RightAngle, J5 Conn_02x03_RightAngle, J6 Conn_02x03_RightAngle

Commit message: HW design progress
Parts:
- renumbered J3 to J10, J6 to J11, J1 to J6, J4 to J7, J2 to J8, J5 to J9

Commit message: hw progress
Parts:
- added C55, C57: 1u, Capacitor_SMD:C_0603_1608Metric, symbol Device:C
- added C56: 10u, Capacitor_SMD:C_0603_1608Metric, symbol Device:C
- added U11: NCP45520, Package_DFN_QFN:DFN-8-1EP_2x2mm_P0.5mm_EP1.05x1.75mm, symbol library:NCP45520
Connections:
- net +5V: now also U11.1 (VIN), U11.9 (VIN); no longer J10.1 (Pin_1), J10.2 (Pin_2), J11.1 (Pin_1), J11.2 (Pin_2), J6.1 (Pin_1), J6.2 (Pin_2), J7.1 (Pin_1), J7.2 (Pin_2), J8.1 (Pin_1), J8.2 (Pin_2), J9.1 (Pin_1), J9.2 (Pin_2)
- net GND: now also C55.2, C56.2, C57.2, U11.4 (GND), U11.6 (PG)
- new net +3V3: C57.1, U11.3 (VCC)
- new net +5V_SW: C55.1, C56.1, J10.1 (Pin_1), J10.2 (Pin_2), J11.1 (Pin_1), J11.2 (Pin_2), J6.1 (Pin_1), J6.2 (Pin_2), J7.1 (Pin_1), J7.2 (Pin_2), J8.1 (Pin_1), J8.2 (Pin_2), J9.1 (Pin_1), J9.2 (Pin_2), U11.5 (BLEED), U11.7 (VOUT), U11.8 (VOUT)
- new net EN: U11.2 (EN)

Commit message: hw progress
Parts:
- added R39: D.N.P., Resistor_SMD:R_0603_1608Metric, symbol Device:R
- J10, J11, J6, J7, J8, J9: footprint Connector_PinHeader_2.54mm:PinHeader_2x03_P2.54mm_Horizontal -> Library:PinHeader_2x03_P2.54mm_Horizontal_SmallSilk
Connections:
- net +5V: now also R39.1
- net +5V_SW: now also R39.2
Changed lines of the file:
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@@
 	(paper "A4")
 	(junction
+		(at 54.61 156.21)
+		(diameter 0)
+		(color 0 0 0 0)
+	)
+	(junction
 		(at 85.09 156.21)
 		(diameter 0)
@@
 	)
 	(junction
+		(at 74.93 156.21)
+		(diameter 0)
+		(color 0 0 0 0)
+	)
+	(junction
 		(at 77.47 156.21)
 		(diameter 0)
@@
 	(wire
 		(pts
+			(xy 54.61 156.21) (xy 54.61 144.78)
+		)
+		(stroke
+			(width 0)
+			(type default)
+		)
+	)
+	(wire
+		(pts
 			(xy 132.08 74.93) (xy 138.43 74.93)
 		)
@@
 	(wire
 		(pts
+			(xy 74.93 144.78) (xy 74.93 156.21)
+		)
+		(stroke
+			(width 0)
+			(type default)
+		)
+	)
+	(wire
+		(pts
 			(xy 97.79 74.93) (xy 91.44 74.93)
 		)
@@
 	(wire
 		(pts
+			(xy 54.61 144.78) (xy 60.96 144.78)
+		)
+		(stroke
+			(width 0)
+			(type default)
+		)
+	)
+	(wire
+		(pts
 			(xy 97.79 115.57) (xy 91.44 115.57)
 		)
@@
 	(wire
 		(pts
+			(xy 68.58 144.78) (xy 74.93 144.78)
+		)
+		(stroke
+			(width 0)
+			(type default)
+		)
+	)
+	(wire
+		(pts
 			(xy 77.47 156.21) (xy 85.09 156.21)
 		)
@@
 			)
 		)
-		(property "Footprint" "Connector_PinHeader_2.54mm:PinHeader_2x03_P2.54mm_Horizontal"
+		(property "Footprint" "Library:PinHeader_2x03_P2.54mm_Horizontal_SmallSilk"
 			(at 208.28 114.3 0)
 			(effects
@@
 			)
 		)
-		(property "Footprint" "Connector_PinHeader_2.54mm:PinHeader_2x03_P2.54mm_Horizontal"
+		(property "Footprint" "Library:PinHeader_2x03_P2.54mm_Horizontal_SmallSilk"
 			(at 83.82 74.93 0)
 			(effects
@@
 			)
 		)
-		(property "Footprint" "Connector_PinHeader_2.54mm:PinHeader_2x03_P2.54mm_Horizontal"
+		(property "Footprint" "Library:PinHeader_2x03_P2.54mm_Horizontal_SmallSilk"
 			(at 143.51 115.57 0)
 			(effects
@@
 	)
 	(symbol
+		(lib_id "Device:R")
+		(at 64.77 144.78 90)
+		(unit 1)
+		(exclude_from_sim no)
+		(in_bom yes)
+		(on_board yes)
+		(dnp no)
+		(property "Reference" "R39"
+			(at 64.77 140.716 90)
+			(effects
+				(font
+					(size 1.27 1.27)
+				)
+			)
+		)
+		(property "Value" "D.N.P."
+			(at 64.77 142.494 90)
+			(effects
+				(font
+					(size 1.27 1.27)
+				)
+			)
+		)
+		(property "Footprint" "Resistor_SMD:R_0603_1608Metric"
+			(at 64.77 146.558 90)
+			(effects
+				(font
+					(size 1.27 1.27)
+				)
+				(hide yes)
+			)
+		)
+		(property "Datasheet" "~"
+			(at 64.77 144.78 0)
+			(effects
+				(font
+					(size 1.27 1.27)
+				)
+				(hide yes)
+			)
+		)
+		(property "Description" "Resistor"
+			(at 64.77 144.78 0)
+			(effects
+				(font
+					(size 1.27 1.27)
+				)
+				(hide yes)
+			)
+		)
+		(pin "1"
+		)
+		(pin "2"
+		)
+		(instances
+			(project "MermaidControlUnit"
+				(path "/613ad2be-9e1b-480a-bebd-92b3f4aa981e/9991d764-5141-439c-a23f-3637534d362c"
+					(reference "R39")
+					(unit 1)
+				)
+			)
+		)
+	)
+	(symbol
 		(lib_id "power:+5V")
 		(at 97.79 67.31 0)
@@
 			)
 		)
-		(property "Footprint" "Connector_PinHeader_2.54mm:PinHeader_2x03_P2.54mm_Horizontal"
+		(property "Footprint" "Library:PinHeader_2x03_P2.54mm_Horizontal_SmallSilk"
 			(at 208.28 76.2 0)
 			(effects
@@
 			)
 		)
-		(property "Footprint" "Connector_PinHeader_2.54mm:PinHeader_2x03_P2.54mm_Horizontal"
+		(property "Footprint" "Library:PinHeader_2x03_P2.54mm_Horizontal_SmallSilk"
 			(at 83.82 115.57 0)
 			(effects
@@
 			)
 		)
-		(property "Footprint" "Connector_PinHeader_2.54mm:PinHeader_2x03_P2.54mm_Horizontal"
+		(property "Footprint" "Library:PinHeader_2x03_P2.54mm_Horizontal_SmallSilk"
 			(at 143.51 74.93 0)
 			(effects

Commit message: production rev A
Parts:
- C55, C57: Part Number (none) -> CL10A105KB8NNNC
- C56: Part Number (none) -> CL10A106MA8NRNC
- J10, J11, J6, J7, J8, J9: Part Number (none) -> BX-PZ2.54-2-3PWZ
- U11: Part Number (none) -> NCP45520IMNTWG-H
Changed lines of the file:
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@@
+			)
+		)
+		(property "Part Number" "BX-PZ2.54-2-3PWZ"
+			(at 208.28 114.3 0)
+			(effects
+				(font
+					(size 1.27 1.27)
+				)
+				(hide yes)
 			)
 		)
@@
 			)
 		)
+		(property "Part Number" "BX-PZ2.54-2-3PWZ"
+			(at 83.82 74.93 0)
+			(effects
+				(font
+					(size 1.27 1.27)
+				)
+				(hide yes)
+			)
+		)
 		(pin "6"
 		)
@@
 			)
 		)
+		(property "Part Number" "BX-PZ2.54-2-3PWZ"
+			(at 143.51 115.57 0)
+			(effects
+				(font
+					(size 1.27 1.27)
+				)
+				(hide yes)
+			)
+		)
 		(pin "6"
 		)
@@
 			)
 		)
+		(property "Part Number" "CL10A106MA8NRNC "
+			(at 90.17 162.56 0)
+			(effects
+				(font
+					(size 1.27 1.27)
+				)
+				(hide yes)
+			)
+		)
 		(pin "2"
 		)
@@
 		)
 		(property "Description" "Unpolarized capacitor"
+			(at 41.91 167.64 0)
+			(effects
+				(font
+					(size 1.27 1.27)
+				)
+				(hide yes)
+			)
+		)
+		(property "Part Number" "CL10A105KB8NNNC "
 			(at 41.91 167.64 0)
 			(effects
@@
 			)
 		)
+		(property "Part Number" "NCP45520IMNTWG-H "
+			(at 64.77 162.56 0)
+			(effects
+				(font
+					(size 1.27 1.27)
+				)
+				(hide yes)
+			)
+		)
 		(pin "6"
 		)
@@
 			)
 		)
+		(property "Part Number" "BX-PZ2.54-2-3PWZ"
+			(at 208.28 76.2 0)
+			(effects
+				(font
+					(size 1.27 1.27)
+				)
+				(hide yes)
+			)
+		)
 		(pin "6"
 		)
@@
 			)
 		)
+		(property "Part Number" "BX-PZ2.54-2-3PWZ"
+			(at 83.82 115.57 0)
+			(effects
+				(font
+					(size 1.27 1.27)
+				)
+				(hide yes)
+			)
+		)
 		(pin "6"
 		)
@@
 			)
 		)
+		(property "Part Number" "BX-PZ2.54-2-3PWZ"
+			(at 143.51 74.93 0)
+			(effects
+				(font
+					(size 1.27 1.27)
+				)
+				(hide yes)
+			)
+		)
 		(pin "6"
 		)
@@
 			(at 85.09 162.56 0)
 			(effects
+				(font
+					(size 1.27 1.27)
+				)
+				(hide yes)
+			)
+		)
+		(property "Part Number" "CL10A105KB8NNNC "
+			(at 85.09 162.56 0)
+			(effects
