File: HW/MermaidControlUnit_A/powering.kicad_sch (KiCad schematic)
At the start: 37 parts, among them Q1 IRLML6244, U2 IP5310, U4 AP2112K-3.3

Commit message: HW design progress
Parts:
- added F1: T5A, Fuse:Fuse_0603_1608Metric, symbol Device:Fuse
- added J4: Batt+, TestPoint:TestPoint_THTPad_2.0x2.0mm_Drill1.0mm, symbol Connector_Generic:Conn_01x01
- added J5: Batt-, TestPoint:TestPoint_THTPad_2.0x2.0mm_Drill1.0mm, symbol Connector_Generic:Conn_01x01
- added R24: D.N.P., Resistor_SMD:R_0603_1608Metric, symbol Device:R
- added TP21, TP22, TP23, TP24, TP25, TP26, TP27, TP28, TP29: TestPoint, TestPoint:TestPoint_Pad_D2.0mm, symbol Connector:TestPoint
- C12: renamed from C9; footprint (none) -> Capacitor_SMD:C_0603_1608Metric
- C13: renamed from C11; footprint (none) -> Capacitor_SMD:C_0603_1608Metric
- C14: renamed from C12; footprint (none) -> Capacitor_SMD:C_0603_1608Metric
- C15: renamed from C10; footprint (none) -> Capacitor_SMD:C_0603_1608Metric
- C16: renamed from C8; footprint (none) -> Capacitor_SMD:C_0603_1608Metric
- C17: renamed from C3; footprint (none) -> Capacitor_SMD:C_0603_1608Metric
- C18: renamed from C7; footprint (none) -> Capacitor_SMD:C_0603_1608Metric
- C19: renamed from C6; footprint (none) -> Capacitor_SMD:C_0603_1608Metric
- C20: renamed from C4; footprint (none) -> Capacitor_SMD:C_0603_1608Metric
- C21: renamed from C5; footprint (none) -> Capacitor_SMD:C_0603_1608Metric
- C22: renamed from C2; footprint (none) -> Capacitor_SMD:C_0603_1608Metric
- C23: renamed from C1; footprint (none) -> Capacitor_SMD:C_0603_1608Metric
- D4: renamed from D1; footprint (none) -> LED_SMD:LED_0603_1608Metric
- D5: renamed from D2; footprint (none) -> LED_SMD:LED_0603_1608Metric
- D6: renamed from D3; footprint (none) -> LED_SMD:LED_0603_1608Metric
- D7: renamed from D4; footprint (none) -> LED_SMD:LED_0603_1608Metric
- L1: footprint (none) -> Inductor_SMD:L_Sunlord_MWSA1204S-1R0; Part Number (none) -> SL1265-1R0M
- R12: renamed from R17; footprint (none) -> Resistor_SMD:R_0603_1608Metric
- R13: renamed from R9; footprint (none) -> Resistor_SMD:R_0603_1608Metric
- R14: renamed from R1; footprint (none) -> Resistor_SMD:R_0603_1608Metric
- R15: renamed from R2; footprint (none) -> Resistor_SMD:R_0603_1608Metric
- R16: renamed from R3; footprint (none) -> Resistor_SMD:R_0603_1608Metric
- R17: renamed from R4; footprint (none) -> Resistor_SMD:R_0603_1608Metric
- R18: renamed from R5; footprint (none) -> Resistor_SMD:R_0603_1608Metric
- R19: renamed from R6; footprint (none) -> Resistor_SMD:R_0603_1608Metric
- R20: renamed from R7; footprint (none) -> Resistor_SMD:R_0603_1608Metric
- R21: renamed from R8; footprint (none) -> Resistor_SMD:R_0603_1608Metric
- R22: renamed from R14; footprint (none) -> Resistor_SMD:R_0603_1608Metric
- R23: renamed from R16; footprint (none) -> Resistor_SMD:R_0603_1608Metric
- R25: renamed from R15; value 47R -> 220R; footprint (none) -> Resistor_SMD:R_0603_1608Metric
- R26: renamed from R10; footprint (none) -> Resistor_SMD:R_0603_1608Metric
- R27: renamed from R11; footprint (none) -> Resistor_SMD:R_0603_1608Metric
- R28: renamed from R12; footprint (none) -> Resistor_SMD:R_0603_1608Metric
- R29: renamed from R13; footprint (none) -> Resistor_SMD:R_0603_1608Metric
- renumbered U4 to U2, U2 to U3
Connections:
- net +3V3: now also TP23.1
- net +5V: now also TP24.1
- net +BATT: now also F1.2, TP22.1
- net GND: now also J5.1 (Pin_1)
- net IRQ: now also TP27.1
- net KEY: now also R24.2
- net LDO_EN: now also TP21.1
- net SCK: now also TP28.1
- net SDA: now also TP29.1
- net at L1.1, U3.14 (LX), U3.15 (LX)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: now also TP25.1
- net at Q1.3 (D), R22.1, U3.8 (KEY): now also R24.1, TP26.1
- new net: F1.1, J4.1 (Pin_1)
- no-connect marks 1 -> 11
Other:
- moved on the sheet: C12, C13, C14, C15, R12, R20, R21, R22, U2

Commit message: hw progress
Parts:
- added C58, C59, C60, C61: 47u, Capacitor_SMD:C_0805_2012Metric, symbol Device:C
- added R38: D.N.P., Resistor_SMD:R_0603_1608Metric, symbol Device:R
- L1: footprint Inductor_SMD:L_Sunlord_MWSA1204S-1R0 -> Inductor_SMD:L_PCC-M1040M-LP; Part Number SL1265-1R0M -> ETQP4M1R0KVC
- TP21, TP22, TP23, TP24, TP25, TP26, TP27, TP28, TP29: footprint TestPoint:TestPoint_Pad_D2.0mm -> TestPoint:TestPoint_Pad_D1.5mm
Connections:
- net +BATT: now also C58.1, C59.1, R38.2
- net +VIN: now also C60.1, C61.1
- net GND: now also C58.2, C59.2, C60.2, C61.2
- net LDO_EN: now also R38.1
Other:
- moved on the sheet: TP22

Commit message: hw progress
Parts:
- R21: Part Number (none) -> NCU18WF104F6SRB
Changed lines of the file:
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@@
+			)
+		)
+		(property "Part Number" "NCU18WF104F6SRB"
+			(at 173.99 111.76 90)
+			(effects
+				(font
+					(size 1.27 1.27)
+				)
+				(hide yes)
 			)
 		)

Commit message: production rev A
Parts:
- C12, C15, C17, C20: Part Number (none) -> CL10A106MA8NRNC
- C13, C14: Part Number (none) -> CL10A105KB8NNNC
- C16, C18, C19, C21, C22, C23: Part Number (none) -> CL10A226MP8NUNE
- C58, C59, C60, C61: Part Number (none) -> GRM21BR61A476ME15L
- D4, D5, D6, D7: value LED -> BLUE; Part Number (none) -> APT1608QBC/D
- F1: Part Number (none) -> F0603HI8000V032TM
- Q1: Part Number (none) -> IRLML6244TRPBF
- R12: Part Number (none) -> RC0603FR-07100KL
- R13: Part Number (none) -> FRC0603F2R00TS
- R14: Part Number (none) -> RC0603FR-070RL
- R20: Part Number (none) -> RC0603FR-0782KL
- R23: Part Number (none) -> RC0603FR-0710KL
- R25: value 220R -> 110R; Part Number (none) -> 0603WAF1100T5E
- R26: Part Number (none) -> RC0603FR-071KL
- U2: Part Number (none) -> AP2112K-3.3TRG1
- U3: footprint Package_DFN_QFN:QFN-32-1EP_5x5mm_P0.5mm_EP3.3x3.3mm_ThermalVias -> Package_DFN_QFN:QFN-32-1EP_5x5mm_P0.5mm_EP3.6x3.6mm_ThermalVias; Part Number (none) -> IP5310
