File: HW/MermaidControlUnit_A/wirelessCharging.kicad_sch (KiCad schematic)
At the start: 0 parts

Commit message: HW design progress
Parts:
- added C36, C37, C38, C43, C44: 10n, Capacitor_SMD:C_0603_1608Metric, symbol Device:C
- added C39, C40, C47, C48, C51, C52: 100n, Capacitor_SMD:C_0603_1608Metric, symbol Device:C
- added C41, C46: 22n, Capacitor_SMD:C_0603_1608Metric, symbol Device:C
- added C42, C45: 470n, Capacitor_SMD:C_0603_1608Metric, symbol Device:C
- added C49, C50, C54: 10u, Capacitor_SMD:C_0603_1608Metric, symbol Device:C
- added C53: 1u, Capacitor_SMD:C_0603_1608Metric, symbol Device:C
- added D8: LED, LED_SMD:LED_0603_1608Metric, symbol Device:LED
- added J12: Coil_1, TestPoint:TestPoint_THTPad_2.0x2.0mm_Drill1.0mm, symbol Connector_Generic:Conn_01x01
- added J13: Coil_2, TestPoint:TestPoint_THTPad_2.0x2.0mm_Drill1.0mm, symbol Connector_Generic:Conn_01x01
- added R30: 1k, Resistor_SMD:R_0603_1608Metric, symbol Device:R
- added R31: 0R, Resistor_SMD:R_0603_1608Metric, symbol Device:R
- added R32: D.N.P., Resistor_SMD:R_0603_1608Metric, symbol Device:R
- added R33: 10k, Resistor_SMD:R_0603_1608Metric, symbol Device:R
- added R34: NTC, Resistor_SMD:R_0603_1608Metric, symbol Device:R
- added R35: 110R, Resistor_SMD:R_0603_1608Metric, symbol Device:R
- added R36: 42.2k, Resistor_SMD:R_0603_1608Metric, symbol Device:R
- added R37: 200R, Resistor_SMD:R_0603_1608Metric, symbol Device:R
- added TP30, TP31, TP32, TP33, TP34, TP35, TP36: TestPoint, TestPoint:TestPoint_Pad_D2.0mm, symbol Connector:TestPoint
- added U10: BQ51013C-Q1, Package_DFN_QFN:Texas_VQFN-RHL-20_ThermalVias, symbol library:BQ51013C-Q1
Connections:
- new net: R35.1, TP32.1, U10.12 (ILIM)
- new net: C51.1, R35.2, R36.2, R37.2, TP35.1, U10.14 (FOD)
- new net: C47.1, R33.2, TP33.1, U10.13 (TS/CTRL)
- new net: C36.1, C37.1, C38.1, J12.1 (Pin_1), TP30.1
- new net: C39.2, C40.2, C44.1, C45.1, C46.1, J13.1 (Pin_1), TP31.1, U10.19 (AC2)
- new net: C44.2, U10.17 (BOOT2)
- new net: D8.1 (K), R30.2
- new net: C36.2, C37.2, C38.2, C39.1, C40.1, C41.1, C42.1, C43.1, U10.2 (AC1)
- new net: C42.2, U10.5 (CLAMP1)
- new net: C45.2, U10.16 (CLAMP2)
- new net: R31.1, R32.1, U10.11 (EN2)
- new net: C46.2, U10.15 (COMM2)
- new net: C48.1, C49.1, C50.1, R36.1, TP34.1, U10.18 (RECT)
- new net: C43.2, U10.3 (BOOT1)
- new net: C41.2, U10.6 (COMM1)
- new net: R30.1, U10.7 (~{CHG})
- new net: R33.1, R34.2
- new net +5V_Charging: C52.1, C53.1, C54.1, D8.2 (A), R32.2, TP36.1, U10.4 (OUT)
- new net GND: C47.2, C48.2, C49.2, C50.2, C51.2, C52.2, C53.2, C54.2, R31.2, R34.1, R37.1, U10.1 (PGND), U10.10 (EN1), U10.20 (PGND), U10.21 (EP), U10.9 (AD)
- no-connect marks 0 -> 1

Commit message: hw progress
Parts:
- TP30, TP31, TP32, TP33, TP34, TP35, TP36: footprint TestPoint:TestPoint_Pad_D2.0mm -> TestPoint:TestPoint_Pad_D1.5mm
Changed lines of the file:
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@@
 			)
 		)
-		(property "Footprint" "TestPoint:TestPoint_Pad_D2.0mm"
+		(property "Footprint" "TestPoint:TestPoint_Pad_D1.5mm"
 			(at 238.76 72.39 0)
 			(effects
@@
 			)
 		)
-		(property "Footprint" "TestPoint:TestPoint_Pad_D2.0mm"
+		(property "Footprint" "TestPoint:TestPoint_Pad_D1.5mm"
 			(at 162.56 88.9 0)
 			(effects
@@
 			)
 		)
-		(property "Footprint" "TestPoint:TestPoint_Pad_D2.0mm"
+		(property "Footprint" "TestPoint:TestPoint_Pad_D1.5mm"
 			(at 59.69 95.25 0)
 			(effects
@@
 			)
 		)
-		(property "Footprint" "TestPoint:TestPoint_Pad_D2.0mm"
+		(property "Footprint" "TestPoint:TestPoint_Pad_D1.5mm"
 			(at 49.53 102.87 0)
 			(effects
@@
 			)
 		)
-		(property "Footprint" "TestPoint:TestPoint_Pad_D2.0mm"
+		(property "Footprint" "TestPoint:TestPoint_Pad_D1.5mm"
 			(at 179.07 113.03 0)
 			(effects
@@
 			)
 		)
-		(property "Footprint" "TestPoint:TestPoint_Pad_D2.0mm"
+		(property "Footprint" "TestPoint:TestPoint_Pad_D1.5mm"
 			(at 201.93 82.55 0)
 			(effects
@@
 			)
 		)
-		(property "Footprint" "TestPoint:TestPoint_Pad_D2.0mm"
+		(property "Footprint" "TestPoint:TestPoint_Pad_D1.5mm"
 			(at 222.25 102.87 0)
 			(effects

Commit message: hw progress
Parts:
- C36: value 10n -> 68n
- C37: value 10n -> 47n
- C38: value 10n -> 39n
- C39: value 100n -> 2n2
- C40: value 100n -> 100p
- R34: value NTC -> NTC 100k; Part Number (none) -> NCU18WF104F6SRB
Other:
- note added: "11.50 uH ± 10%"
- note added: "175.00 mΩ"
- note added: "TCOLD = -10°C THOT = 100°C"
- note added: "YX-A11-R431231-G3232"
- note added: "all C min 25Vrating"
Changed lines of the file:
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@@
+		)
+	)
+	(text "175.00 mΩ"
+		(exclude_from_sim no)
+		(at 33.528 111.506 0)
+		(effects
+			(font
+				(size 1.27 1.27)
+			)
+		)
+	)
+	(text "all C min 25Vrating"
+		(exclude_from_sim no)
+		(at 91.186 116.84 0)
+		(effects
+			(font
+				(size 1.27 1.27)
+			)
+		)
+	)
+	(text "11.50 uH ± 10%"
+		(exclude_from_sim no)
+		(at 36.322 109.22 0)
+		(effects
+			(font
+				(size 1.27 1.27)
+			)
+		)
+	)
+	(text "YX-A11-R431231-G3232"
+		(exclude_from_sim no)
+		(at 40.64 106.934 0)
+		(effects
+			(font
+				(size 1.27 1.27)
+			)
+		)
+	)
+	(text "TCOLD = -10°C\nTHOT = 100°C"
+		(exclude_from_sim no)
+		(at 179.07 137.414 0)
+		(effects
+			(font
+				(size 1.27 1.27)
+			)
 		)
 	)
@@
 			)
 		)
-		(property "Value" "10n"
+		(property "Value" "68n"
 			(at 85.598 86.868 90)
 			(effects
@@
 			)
 		)
-		(property "Value" "100n"
+		(property "Value" "100p"
 			(at 100.33 101.6 0)
 			(effects
@@
 			)
 		)
-		(property "Value" "NTC"
-			(at 169.418 129.54 0)
+		(property "Value" "NTC 100k"
+			(at 163.322 132.334 0)
 			(effects
 				(font
@@
 		)
 		(property "Description" "Resistor"
+			(at 167.64 128.27 0)
+			(effects
+				(font
+					(size 1.27 1.27)
+				)
+				(hide yes)
+			)
+		)
+		(property "Part Number" "NCU18WF104F6SRB"
 			(at 167.64 128.27 0)
 			(effects
@@
 			)
 		)
-		(property "Value" "10n"
+		(property "Value" "39n"
 			(at 85.598 97.028 90)
 			(effects
@@
 			)
 		)
-		(property "Value" "10n"
+		(property "Value" "47n"
 			(at 85.598 91.948 90)
 			(effects
@@
 			)
 		)
-		(property "Value" "100n"
+		(property "Value" "2n2"
 			(at 93.98 101.6 0)
 			(effects

Commit message: production rev A
Parts:
- added R40: 30k, Resistor_SMD:R_0603_1608Metric, symbol Device:R
- C36: Part Number (none) -> GCJ188R71H683KA12D
- C37: Part Number (none) -> CGA3E2X7R1H473KT0Y0N
- C38: Part Number (none) -> CL10B393KB8NNNC
- C39: Part Number (none) -> GRM1885C2A222JA01D
- C40: Part Number (none) -> CGA3E2C0G1H101JT0Y0N
- C41, C46: Part Number (none) -> C1608X7R1H223KT000N
- C42, C45: Part Number (none) -> CL10B474KB8VPNC
- C43, C44: Part Number (none) -> 06035C103JAT2A
- C47, C48, C51, C52: Part Number (none) -> CC0603KRX7R9BB104
- C49, C50, C54: Part Number (none) -> CL10A106MA8NRNC
- C53: Part Number (none) -> CL10A105KB8NNNC
- D8: value LED -> RED; Part Number (none) -> APT1608EC
- R30: Part Number (none) -> RC0603FR-071KL
- R31: Part Number (none) -> RC0603FR-070RL
- R33: value 10k -> 110R; Part Number (none) -> 0603WAF1100T5E
- R35: Part Number (none) -> 0603WAF1100T5E
- R36: Part Number (none) -> WR06X4222FTL
- R37: Part Number (none) -> 0603WAF2000T5E
- U10: Part Number (none) -> BQ51013C-Q1
Connections:
- net GND: now also R40.1
- net at C47.1, R33.2, TP33.1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: now also R40.2
Other:
- note added: "TCOLD = -6°C THOT = 100°C"
- note removed: "TCOLD = -10°C THOT = 100°C"
- note removed: "all C min 25Vrating"
- moved on the sheet: C47, TP33
