File: HW/MermaidControlUnit_A/KiCAD_Project/STM32.kicad_sch (KiCad schematic)
At the start: 36 parts, among them J1 Conn_01x05, J2 Conn_01x03, J3 Conn_01x03, U1 STM32F103CBTx, Y1 ABM3-8.000MHZ-D2Y-T, Y2 CM315D

Commit message: schematic added, folder structure updated
Other:
- note added: "IR Receiver"
- note added: "Programming"
- note added: "UART"
- company: (none) -> Aurora Dreams Mermaids
- title: (none) -> Mermaid Control Unit
Changed lines of the file:
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@@
 	(generator_version "8.0")
 	(paper "A4")
+	(title_block
+		(title "Mermaid Control Unit")
+		(date "2025-02-04")
+		(rev "A")
+		(company "Aurora Dreams Mermaids")
+		(comment 1 "Designed by: Ondrej Ruzicka")
+		(comment 4 "STM32 MCU")
+	)
 	(junction
 		(at 181.61 62.23)
@@
 		)
 	)
+	(text "Programming"
+		(exclude_from_sim no)
+		(at 251.206 103.378 0)
+		(effects
+			(font
+				(size 1.27 1.27)
+			)
+		)
+	)
+	(text "UART"
+		(exclude_from_sim no)
+		(at 251.206 126.746 0)
+		(effects
+			(font
+				(size 1.27 1.27)
+			)
+		)
+	)
+	(text "IR Receiver"
+		(exclude_from_sim no)
+		(at 254.508 27.94 0)
+		(effects
+			(font
+				(size 1.27 1.27)
+			)
+		)
+	)
