File: HW/MermaidControlUnit_A/KiCAD_Project/levelShifter.kicad_sch (KiCad schematic)
At the start: 18 parts, among them U4 SN74LVC2T45DCTR, U5 SN74LVC2T45DCTR, U6 SN74LVC2T45DCTR, U7 SN74LVC2T45DCTR, U8 SN74LVC2T45DCTR, U9 SN74LVC2T45DCTR

Commit message: schematic added, folder structure updated
Other:
- company: (none) -> Aurora Dreams Mermaids
- title: (none) -> Mermaid Control Unit
Changed lines of the file:
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@@
 	(generator_version "8.0")
 	(paper "A4")
+	(title_block
+		(title "Mermaid Control Unit")
+		(date "2025-02-04")
+		(rev "A")
+		(company "Aurora Dreams Mermaids")
+		(comment 1 "Designed by: Ondrej Ruzicka")
+		(comment 4 "Level Shifters")
+	)
 	(junction
 		(at 142.24 39.37)
