File: HW/MermaidControlUnit_A/KiCAD_Project/outputs.kicad_sch (KiCad schematic)
At the start: 11 parts, among them J10 Conn_02x03_RightAngle, J11 Conn_02x03_RightAngle, J6 Conn_02x03_RightAngle, J7 Conn_02x03_RightAngle, J8 Conn_02x03_RightAngle, J9 Conn_02x03_RightAngle, U11 NCP45520

Commit message: schematic added, folder structure updated
Other:
- company: (none) -> Aurora Dreams Mermaids
- title: (none) -> Mermaid Control Unit
Changed lines of the file:
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@@
 	(generator_version "8.0")
 	(paper "A4")
+	(title_block
+		(title "Mermaid Control Unit")
+		(date "2025-02-04")
+		(rev "A")
+		(company "Aurora Dreams Mermaids")
+		(comment 1 "Designed by: Ondrej Ruzicka")
+		(comment 4 "Outputs")
+	)
 	(junction
 		(at 54.61 156.21)
