File: HW/MermaidControlUnit_A/KiCAD_Project/powering.kicad_sch (KiCad schematic)
At the start: 55 parts, among them J4 Batt+, J5 Batt-, Q1 IRLML6244, U2 AP2112K-3.3, U3 IP5310

Commit message: schematic added, folder structure updated
Other:
- company: (none) -> Aurora Dreams Mermaids
- title: (none) -> Mermaid Control Unit
Changed lines of the file:
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@@
 	(generator_version "8.0")
 	(paper "A4")
+	(title_block
+		(title "Mermaid Control Unit")
+		(date "2025-02-04")
+		(rev "A")
+		(company "Aurora Dreams Mermaids")
+		(comment 1 "Designed by: Ondrej Ruzicka")
+		(comment 4 "Powering")
+	)
 	(junction
 		(at 148.59 127)
