File: HW/MermaidControlUnit_A/KiCAD_Project/MermaidControlUnit.kicad_pcb (KiCad board)
At the start: 2 copper layers, 78.1 x 69 mm, 175 parts, among them J1 Conn_01x05, J10 Conn_02x03_RightAngle, J11 Conn_02x03_RightAngle, J12 Coil_1, J13 Coil_2, J2 Conn_01x03, J3 Conn_01x03, J4 Batt+, J5 Batt-, J6 Conn_02x03_RightAngle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

Commit message: BQ NTC retuned
Parts:
- R33: value 110R -> 3.4k
- R34: value NTC 100k -> NTC 10k
- R40: value 30k -> 62k
Changed lines of the file:
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@@
 			)
 		)
-		(property "Value" "NTC 100k"
+		(property "Value" "NTC 10k"
 			(at 0 1.43 0)
 			(layer "F.Fab")
@@
 			)
 		)
-		(property "Part Number" "NCU18WF104F6SRB"
+		(property "Part Number" "NTCG163JF103FTDS"
 			(at 0 0 0)
 			(unlocked yes)
@@
 			)
 		)
-		(property "Value" "30k"
+		(property "Value" "62k"
 			(at 0 1.43 0)
 			(layer "F.Fab")
@@
 			)
 		)
-		(property "Part Number" "0603WAF3002T5E "
+		(property "Part Number" "0603WAF6202T5E  "
 			(at 0 0 180)
 			(unlocked yes)
@@
 			)
 		)
-		(property "Value" "110R"
+		(property "Value" "3.4k"
 			(at 0 1.43 0)
 			(layer "F.Fab")
@@
 			)
 		)
-		(property "Part Number" "0603WAF1100T5E "
+		(property "Part Number" "0603WAF4301T5E  "
 			(at 0 0 180)
 			(unlocked yes)
